File: clkgen/pcb/clkgen.kicad_sch (KiCad schematic)
At the start: 21 parts, among them J1 AudioJack2_SwitchT, J2 AudioJack2_SwitchT, J3 AudioJack2_SwitchT, J4 AudioJack2_SwitchT, J5 AudioJack2_SwitchT, J6 EurorackPwr, U1 4521

Commit message: first pcb layout
Parts:
- C1, C2, C3, C4: footprint (none) -> Capacitor_SMD:C_0603_1608Metric
- D1, D2: footprint (none) -> Diode_SMD:D_SOD-123
- J1, J2, J3, J4, J5: footprint (none) -> eurorack_footprints:audio_jack_pj-398sm
- J6: footprint (none) -> Connector_PinHeader_2.54mm:PinHeader_2x05_P2.54mm_Vertical
- R1, R2, R3, R4, R5, R6, R7: footprint (none) -> Resistor_SMD:R_0603_1608Metric
- RV1: footprint (none) -> eurorack_footprints:pot1_B
- U1: footprint (none) -> Package_SO:SOIC-16_3.9x9.9mm_P1.27mm
