File: att_x2_mult_1x4/panel/att_x2_mult_1x4_face.kicad_pcb (KiCad board)
At the start: 2 copper layers, 20 x 128.5 mm, 12 parts

Commit message: moved resistor, added scale to panel
Changed lines of the file:
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@@
   )
   (gr_line (start 104.14 134.62) (end 114.3 134.62) (layer "F.SilkS") (width 0.5))
+  (gr_arc (start 102.87 71.12) (mid 109.474 55.59895) (end 116.078 71.12) (layer "F.SilkS") (width 0.5))
+  (gr_line (start 100.076 86.36) (end 118.11 86.36) (layer "F.SilkS") (width 0.5))
+  (gr_line (start 113.03 104.14) (end 116.078 104.14) (layer "F.SilkS") (width 0.5))
   (gr_line (start 104.14 134.62) (end 104.14 147.32) (layer "F.SilkS") (width 0.5))
+  (gr_line (start 102.87 71.12) (end 101.6 68.58) (layer "F.SilkS") (width 0.5))
+  (gr_arc (start 102.87 104.14) (mid 109.474 88.61895) (end 116.078 104.14) (layer "F.SilkS") (width 0.5))
+  (gr_line (start 102.87 104.14) (end 101.6 101.6) (layer "F.SilkS") (width 0.5))
+  (gr_arc (start 101.6 68.58) (mid 109.880285 58.306216) (end 113.03 71.12) (layer "F.SilkS") (width 0.5))
+  (gr_line (start 100.33 119.38) (end 118.364 119.38) (layer "F.SilkS") (width 0.5))
   (gr_line (start 104.14 147.32) (end 114.3 147.32) (layer "F.SilkS") (width 0.5))
   (gr_line (start 114.3 134.62) (end 114.3 147.32) (layer "F.SilkS") (width 0.5))
-  (gr_text "OUT" (at 114.3 88.265) (layer "F.SilkS")
+  (gr_arc (start 101.6 101.6) (mid 109.880285 91.326216) (end 113.03 104.14) (layer "F.SilkS") (width 0.5))
+  (gr_line (start 113.03 71.12) (end 116.078 71.12) (layer "F.SilkS") (width 0.5))
+  (gr_text "OUT" (at 114.3 76.2) (layer "F.SilkS")
     (effects (font (size 2 2) (thickness 0.15)))
   )
-  (gr_text "OUT" (at 114.3 121.285) (layer "F.SilkS")
+  (gr_text "OUT" (at 114.3 109.22) (layer "F.SilkS")
     (effects (font (size 2 2) (thickness 0.15)))
   )
-  (gr_text "IN" (at 104.14 121.285) (layer "F.SilkS")
+  (gr_text "IN" (at 104.14 109.22) (layer "F.SilkS")
     (effects (font (size 2 2) (thickness 0.15)))
   )
@@
     (effects (font (size 2.5 2.5) (thickness 0.5)))
   )
-  (gr_text "IN" (at 104.14 88.265) (layer "F.SilkS")
+  (gr_text "IN" (at 104.14 76.2) (layer "F.SilkS")
     (effects (font (size 2 2) (thickness 0.15)))
   )

Commit message: modified ring
Parts:
- removed the G*** at (109.1, 161.9)
- added G***: LOGO, eurorack_footprints:musikbeton_10mm_front, F.Cu at (109.1, 161.9)
- moved REF** 2.54 mm to (114.3, 149.9)
- moved REF** 2.54 mm to (104.1, 149.9)
- moved REF** 2.54 mm to (114.3, 116.8)
- moved REF** 2.54 mm to (104.1, 116.8)
- moved REF** 2.54 mm to (109.2, 67.3)
- moved REF** 2.54 mm to (114.3, 83.8)
- moved REF** 2.54 mm to (109.2, 100.3)
- moved REF** 2.54 mm to (104.1, 137.2)
- moved REF** 2.54 mm to (104.1, 83.8)
- moved REF** 2.54 mm to (114.3, 137.2)

Commit message: extended mult to 2x3
Parts:
- removed the REF** at (114.3, 149.9)
- removed the REF** at (104.1, 137.2)
- removed the REF** at (104.1, 149.9)
- removed the REF** at (114.3, 137.2)
- added REF**: panel_jackhole, eurorack_footprints:panel_jackhole, B.Cu at (104.1, 129.4)
- added REF**1: panel_jackhole, eurorack_footprints:panel_jackhole, B.Cu at (114.3, 129.4)
- added REF**2: panel_jackhole, eurorack_footprints:panel_jackhole, B.Cu at (104.1, 142.1)
- added REF**3: panel_jackhole, eurorack_footprints:panel_jackhole, B.Cu at (114.3, 142.1)
- added REF**4: panel_jackhole, eurorack_footprints:panel_jackhole, B.Cu at (104.1, 154.8)
- added REF**5: panel_jackhole, eurorack_footprints:panel_jackhole, B.Cu at (114.3, 154.8)
- moved REF** 2.54 mm to (109.2, 64.8)
- moved REF** 2.54 mm to (114.3, 81.3)
- moved REF** 2.54 mm to (104.1, 81.3)
- moved REF** 1.54 mm to (114.3, 115.3)
- moved REF** 1.54 mm to (104.1, 115.3)
- moved REF** 1.54 mm to (109.2, 98.8)

Commit message: revert cheanges on pat
Parts:
- removed the REF** at (104.1, 129.4)
- removed REF**1, REF**2, REF**3, REF**4, REF**5: panel_jackhole, eurorack_footprints:panel_jackhole
- added REF**: panel_jackhole, eurorack_footprints:panel_jackhole, F.Cu at (114.3, 149.9)
- added REF**: panel_jackhole, eurorack_footprints:panel_jackhole, F.Cu at (104.1, 137.2)
- added REF**: panel_jackhole, eurorack_footprints:panel_jackhole, F.Cu at (104.1, 149.9)
- added REF**: panel_jackhole, eurorack_footprints:panel_jackhole, F.Cu at (114.3, 137.2)
- moved REF** 2.54 mm to (109.2, 67.3)
- moved REF** 2.54 mm to (114.3, 83.8)
- moved REF** 2.54 mm to (104.1, 83.8)
- moved REF** 1.54 mm to (114.3, 116.8)
- moved REF** 1.54 mm to (104.1, 116.8)
- moved REF** 1.54 mm to (109.2, 100.3)

Commit message: moved second attenuator slightly down
Parts:
- moved REF** 2.54 mm to (109.2, 102.9)
- moved REF** 2.54 mm to (114.3, 119.4)
- moved REF** 2.54 mm to (104.1, 119.4)
Changed lines of the file:
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@@
   )
   (footprint "eurorack_footprints:panel_jackhole" (layer "F.Cu")
-    (at 114.3 116.84)
+    (at 114.3 119.38)
     (attr smd)
     (fp_text reference "REF**" (at 0 -0.5 unlocked) (layer "F.SilkS") hide
@@
   )
   (footprint "eurorack_footprints:panel_jackhole" (layer "F.Cu")
-    (at 104.14 116.84)
+    (at 104.14 119.38)
     (attr smd)
     (fp_text reference "REF**" (at 0 -0.5 unlocked) (layer "F.SilkS") hide
@@
   )
   (footprint "eurorack_footprints:panel_pothole" (layer "F.Cu")
-    (at 109.22 100.33)
+    (at 109.22 102.87)
     (attr smd)
     (fp_text reference "REF**" (at 0 -0.5 unlocked) (layer "F.SilkS") hide
@@
   )
   (gr_line (start 104.14 137.16) (end 114.3 137.16) (layer "F.SilkS") (width 0.5))
-  (gr_line (start 112.395 107.95) (end 114.935 107.95) (layer "F.SilkS") (width 0.5))
+  (gr_line (start 112.395 110.49) (end 114.935 110.49) (layer "F.SilkS") (width 0.5))
   (gr_arc (start 103.505 74.93) (mid 109.22 58.596215) (end 114.935 74.93) (layer "F.SilkS") (width 0.5))
-  (gr_line (start 100.076 88.9) (end 118.11 88.9) (layer "F.SilkS") (width 0.5))
+  (gr_line (start 101.3648 90.17) (end 116.745 90.17) (layer "F.SilkS") (width 0.5))
   (gr_line (start 104.14 137.16) (end 104.14 149.86) (layer "F.SilkS") (width 0.5))
   (gr_line (start 103.505 74.93) (end 102.235 72.39) (layer "F.SilkS") (width 0.5))
-  (gr_line (start 103.505 107.95) (end 102.235 105.41) (layer "F.SilkS") (width 0.5))
+  (gr_line (start 103.505 110.49) (end 102.235 107.95) (layer "F.SilkS") (width 0.5))
   (gr_arc (start 102.235 72.39) (mid 110.532136 60.791451) (end 112.395 74.93) (layer "F.SilkS") (width 0.5))
-  (gr_line (start 100.33 121.92) (end 118.364 121.92) (layer "F.SilkS") (width 0.5))
-  (gr_arc (start 102.235 105.41) (mid 110.532136 93.811451) (end 112.395 107.95) (layer "F.SilkS") (width 0.5))
+  (gr_arc (start 102.235 107.95) (mid 110.532145 96.35142) (end 112.395 110.49) (layer "F.SilkS") (width 0.5))
   (gr_line (start 104.14 149.86) (end 114.3 149.86) (layer "F.SilkS") (width 0.5))
-  (gr_arc (start 103.505 107.95) (mid 109.22 91.616215) (end 114.935 107.95) (layer "F.SilkS") (width 0.5))
+  (gr_arc (start 103.505 110.49) (mid 109.22 94.156215) (end 114.935 110.49) (layer "F.SilkS") (width 0.5))
   (gr_line (start 114.3 137.16) (end 114.3 149.86) (layer "F.SilkS") (width 0.5))
+  (gr_line (start 101.3648 128.17) (end 116.745 128.17) (layer "F.SilkS") (width 0.5))
   (gr_line (start 112.395 74.93) (end 114.935 74.93) (layer "F.SilkS") (width 0.5))
   (gr_text "OUT" (at 114.3 78.74) (layer "F.SilkS")
     (effects (font (size 2 2) (thickness 0.15)))
   )
-  (gr_text "OUT" (at 114.3 111.76) (layer "F.SilkS")
+  (gr_text "OUT" (at 114.3 114.3) (layer "F.SilkS")
     (effects (font (size 2 2) (thickness 0.15)))
   )
-  (gr_text "IN" (at 104.14 111.76) (layer "F.SilkS")
+  (gr_text "IN" (at 104.14 114.3) (layer "F.SilkS")
     (effects (font (size 2 2) (thickness 0.15)))
   )
