File: att_x2_mult_1x4/pcb/att_x2_mult_1x4.kicad_sch (KiCad schematic)
At the start: 12 parts, among them J1 AudioJack2_SwitchT, J2 AudioJack2_SwitchT, J3 AudioJack2_SwitchT, J4 AudioJack2_SwitchT, J5 AudioJack2_SwitchT, J6 AudioJack2_SwitchT, J7 AudioJack2_SwitchT, J8 AudioJack2_SwitchT

Commit message: replaced tht resistor with an smd
Parts:
- R1, R2: footprint Resistor_THT:R_Axial_DIN0309_L9.0mm_D3.2mm_P12.70mm_Horizontal -> Resistor_SMD:R_0805_2012Metric
Changed lines of the file:
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@@
     (property "Reference" "R1" (id 0) (at 99.06 72.39 90))
     (property "Value" "1k" (id 1) (at 93.98 72.39 90))
-    (property "Footprint" "Resistor_THT:R_Axial_DIN0309_L9.0mm_D3.2mm_P12.70mm_Horizontal" (id 2) (at 96.52 68.072 90)
+    (property "Footprint" "Resistor_SMD:R_0805_2012Metric" (id 2) (at 96.52 68.072 90)
       (effects (font (size 1.27 1.27)) hide)
     )
@@
     (property "Reference" "R2" (id 0) (at 186.69 72.39 90))
     (property "Value" "1k" (id 1) (at 181.61 72.39 90))
-    (property "Footprint" "Resistor_THT:R_Axial_DIN0309_L9.0mm_D3.2mm_P12.70mm_Horizontal" (id 2) (at 184.15 68.072 90)
+    (property "Footprint" "Resistor_SMD:R_0805_2012Metric" (id 2) (at 184.15 68.072 90)
       (effects (font (size 1.27 1.27)) hide)
     )
@@
     )
     (path "/1868205c-ee30-4243-a4a5-3b8be43dc87c"
-      (reference "R1") (unit 1) (value "1k") (footprint "Resistor_THT:R_Axial_DIN0309_L9.0mm_D3.2mm_P12.70mm_Horizontal")
+      (reference "R1") (unit 1) (value "1k") (footprint "Resistor_SMD:R_0805_2012Metric")
     )
     (path "/918a10d6-bd6e-4091-a5c1-2b6426167538"
-      (reference "R2") (unit 1) (value "1k") (footprint "Resistor_THT:R_Axial_DIN0309_L9.0mm_D3.2mm_P12.70mm_Horizontal")
+      (reference "R2") (unit 1) (value "1k") (footprint "Resistor_SMD:R_0805_2012Metric")
     )
     (path "/6a01f3f0-dee7-4458-934b-b9d2961ad3ec"

Commit message: updated pot footprint, changed rout back to tht
Parts:
- R1, R2: footprint Resistor_SMD:R_0805_2012Metric -> Resistor_THT:R_Axial_DIN0207_L6.3mm_D2.5mm_P10.16mm_Horizontal
Changed lines of the file:
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@@
     (property "Reference" "R1" (id 0) (at 99.06 72.39 90))
     (property "Value" "1k" (id 1) (at 93.98 72.39 90))
-    (property "Footprint" "Resistor_SMD:R_0805_2012Metric" (id 2) (at 96.52 68.072 90)
+    (property "Footprint" "Resistor_THT:R_Axial_DIN0207_L6.3mm_D2.5mm_P10.16mm_Horizontal" (id 2) (at 96.52 68.072 90)
       (effects (font (size 1.27 1.27)) hide)
     )
@@
     (property "Reference" "R2" (id 0) (at 186.69 72.39 90))
     (property "Value" "1k" (id 1) (at 181.61 72.39 90))
-    (property "Footprint" "Resistor_SMD:R_0805_2012Metric" (id 2) (at 184.15 68.072 90)
+    (property "Footprint" "Resistor_THT:R_Axial_DIN0207_L6.3mm_D2.5mm_P10.16mm_Horizontal" (id 2) (at 184.15 68.072 90)
       (effects (font (size 1.27 1.27)) hide)
     )
@@
     )
     (path "/1868205c-ee30-4243-a4a5-3b8be43dc87c"
-      (reference "R1") (unit 1) (value "1k") (footprint "Resistor_SMD:R_0805_2012Metric")
+      (reference "R1") (unit 1) (value "1k") (footprint "Resistor_THT:R_Axial_DIN0207_L6.3mm_D2.5mm_P10.16mm_Horizontal")
     )
     (path "/918a10d6-bd6e-4091-a5c1-2b6426167538"
-      (reference "R2") (unit 1) (value "1k") (footprint "Resistor_SMD:R_0805_2012Metric")
+      (reference "R2") (unit 1) (value "1k") (footprint "Resistor_THT:R_Axial_DIN0207_L6.3mm_D2.5mm_P10.16mm_Horizontal")
     )
     (path "/6a01f3f0-dee7-4458-934b-b9d2961ad3ec"

Commit message: reverted panel ; change pot direction
Parts:
- RV1, RV2: footprint eurorack_footprints:pot1_A -> eurorack_footprints:pot1_B
Changed lines of the file:
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@@
       (effects (font (size 1.27 1.27)) (justify right))
     )
-    (property "Footprint" "eurorack_footprints:pot1_A" (id 2) (at 104.14 62.23 0)
+    (property "Footprint" "eurorack_footprints:pot1_B" (id 2) (at 104.14 62.23 0)
       (effects (font (size 1.27 1.27)) hide)
     )
@@
       (effects (font (size 1.27 1.27)) (justify right))
     )
-    (property "Footprint" "eurorack_footprints:pot1_A" (id 2) (at 191.77 62.23 0)
+    (property "Footprint" "eurorack_footprints:pot1_B" (id 2) (at 191.77 62.23 0)
       (effects (font (size 1.27 1.27)) hide)
     )
@@
     )
     (path "/6a01f3f0-dee7-4458-934b-b9d2961ad3ec"
-      (reference "RV1") (unit 1) (value "100k") (footprint "eurorack_footprints:pot1_A")
+      (reference "RV1") (unit 1) (value "100k") (footprint "eurorack_footprints:pot1_B")
     )
     (path "/f7b36b53-34c7-4607-bce1-aa12ccdeb5a8"
-      (reference "RV2") (unit 1) (value "100k") (footprint "eurorack_footprints:pot1_A")
+      (reference "RV2") (unit 1) (value "100k") (footprint "eurorack_footprints:pot1_B")
     )
   )
